Commit message: Fixed odometry, made main smarter

File: src/orc/robot.urdf (robot description, URDF)
Before this commit: robot GLaDOS, 6 links, 5 joints
Links:
- link gripper: geometry collision box size=0.12 0.02 0.02; visual box size=0.12 0.02 0.02
- link left_wheel: geometry collision cylinder length=0.02 radius=0.0625; visual cylinder length=0.02 radius=0.0625
- link right_wheel: geometry collision cylinder length=0.02 radius=0.0625; visual cylinder length=0.02 radius=0.0625
- link shoulder: geometry collision box size=0.02 0.02 0.244; visual box size=0.02 0.02 0.244
- link wrist: geometry collision box size=0.065 0.02 0.02; visual box size=0.065 0.02 0.02

Commit message: Bunch of stuff

File: src/orc/robot.urdf (robot description, URDF)
Before this commit: robot GLaDOS, 6 links, 5 joints
Links:
- added link camera_base; visual box size=0.1 0.3 0.03
- added link camera_link
Joints:
- added joint base_to_camera: type fixed, parent base_link, child camera_base, origin xyz=-0.1143 -0.1524 0.4 rpy=0 0.698131701 0
- added joint camera_base_to_camera_link: type fixed, parent camera_base, child camera_link, origin xyz=-0.018 0 0

Commit message: Changes to the location of the kinect

File: src/orc/robot.urdf (robot description, URDF)
Before this commit: robot GLaDOS, 8 links, 7 joints
Links:
- link gripper: geometry visual box size=0.12 0.02 0.02
- link shoulder: geometry visual box size=0.02 0.02 0.244
- link wrist: geometry visual box size=0.065 0.02 0.02
Joints:
- joint base_to_camera: origin xyz=-0.1143 -0.1524 0.4 rpy=0 0.698131701 0 -> xyz=-0.1143 -0.1778 0.4 rpy=0 0.698131701 0
